File: SIM28M/SIM28M.kicad_pcb (KiCad board)
At the start: 2 copper layers, 22.7 x 20.3 mm, 25 parts, among them J1 Conn_01x05, J2 Conn_01x05, U2 AP7365-W-7

Commit message: Layout Updated
Parts:
- added JP1: SolderJumper_2_Open, Jumper:SolderJumper-2_P1.3mm_Open_RoundedPad1.0x1.5mm, B.Cu at (54.8, 40.5)
- renumbered GPS to AE1, BT1 to CR1220, SirBoard to SIM28M
Connections:
- L1 pad 1: Net-(AE1-Pad1) -> Net-(JP1-Pad1)
Routing:
- net Net-(JP1-Pad1): track 0.00 -> 4.10 mm, vias 0 -> 1
- net VBAT: track 28.8 -> 31.6 mm
- net Net-(AE1-Pad1): track 5.58 -> 5.93 mm, vias 0 -> 1
Other:
- board text added: "SIM28M www.SirBoard.com"
Changed lines of the file:
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@@
   (general
     (thickness 1.6)
-    (drawings 25)
-    (tracks 106)
+    (drawings 26)
+    (tracks 117)
     (zones 0)
-    (modules 25)
-    (nets 24)
+    (modules 26)
+    (nets 25)
   )
   (page User 132.004 102.006)
@@
   (net 22 TXD0)
   (net 23 VBAT)
+  (net 24 "Net-(JP1-Pad1)")
   (net_class Default "This is the default net class."
     (clearance 0.127)
@@
     (add_net "Net-(IC1-Pad7)")
     (add_net "Net-(IC1-Pad9)")
+    (add_net "Net-(JP1-Pad1)")
     (add_net "Net-(L1-Pad2)")
     (add_net "Net-(R7-Pad2)")
@@
     (add_net VIN)
   )
+  (module MountingHole:MountingHole_2.7mm_M2.5_ISO14580_Pad (layer F.Cu)
+    (at 54.61 44.45 270)
+    (descr "Mounting Hole 2.7mm, M2.5, ISO14580")
+    (tags "mounting hole 2.7mm m2.5 iso14580")
+    (attr virtual)
+    (fp_text reference H1 (at 0 0 90) (layer F.SilkS) hide
+      (effects (font (size 1 1) (thickness 0.15)))
+    )
+    (fp_text value MountingHole (at 0 3.25 90) (layer F.Fab)
+      (effects (font (size 1 1) (thickness 0.15)))
+    )
+    (fp_circle (center 0 0) (end 2.5 0) (layer F.CrtYd) (width 0.05))
+    (fp_circle (center 0 0) (end 2.25 0) (layer Cmts.User) (width 0.15))
+    (fp_text user %R (at 0.3 0 90) (layer F.Fab)
+      (effects (font (size 1 1) (thickness 0.15)))
+    )
+    (pad 1 thru_hole circle (at 0 0 270) (size 4.5 4.5) (drill 2.7) (layers *.Cu *.Mask))
+  )
+  (module Jumper:SolderJumper-2_P1.3mm_Open_RoundedPad1.0x1.5mm (layer B.Cu)
+    (at 54.8005 40.513)
+    (descr "SMD Solder Jumper, 1x1.5mm, rounded Pads, 0.3mm gap, open")
+    (tags "solder jumper open")
+    (attr virtual)
+    (fp_text reference JP1 (at 0 1.8) (layer B.SilkS) hide
+      (effects (font (size 1 1) (thickness 0.15)) (justify mirror))
+    )
+    (fp_text value SolderJumper_2_Open (at 0 -1.9) (layer B.Fab)
+      (effects (font (size 1 1) (thickness 0.15)) (justify mirror))
+    )
+    (fp_line (start 1.65 -1.25) (end -1.65 -1.25) (layer B.CrtYd) (width 0.05))
+    (fp_line (start 1.65 -1.25) (end 1.65 1.25) (layer B.CrtYd) (width 0.05))
+    (fp_line (start -1.65 1.25) (end -1.65 -1.25) (layer B.CrtYd) (width 0.05))
+    (fp_line (start -1.65 1.25) (end 1.65 1.25) (layer B.CrtYd) (width 0.05))
+    (fp_line (start -0.7 1) (end 0.7 1) (layer B.SilkS) (width 0.12))
+    (fp_line (start 1.4 0.3) (end 1.4 -0.3) (layer B.SilkS) (width 0.12))
+    (fp_line (start 0.7 -1) (end -0.7 -1) (layer B.SilkS) (width 0.12))
+    (fp_line (start -1.4 -0.3) (end -1.4 0.3) (layer B.SilkS) (width 0.12))
+    (fp_arc (start -0.7 0.3) (end -0.7 1) (angle 90) (layer B.SilkS) (width 0.12))
+    (fp_arc (start -0.7 -0.3) (end -1.4 -0.3) (angle 90) (layer B.SilkS) (width 0.12))
+    (fp_arc (start 0.7 -0.3) (end 0.7 -1) (angle 90) (layer B.SilkS) (width 0.12))
+    (fp_arc (start 0.7 0.3) (end 1.4 0.3) (angle 90) (layer B.SilkS) (width 0.12))
+    (pad 2 smd custom (at 0.65 0) (size 1 0.5) (layers B.Cu B.Mask)
+      (net 6 "Net-(AE1-Pad1)") (zone_connect 2)
+      (options (clearance outline) (anchor rect))
+      (primitives
+        (gr_circle (center 0 -0.25) (end 0.5 -0.25) (width 0))
+        (gr_circle (center 0 0.25) (end 0.5 0.25) (width 0))
+        (gr_poly (pts
+           (xy 0 0.75) (xy -0.5 0.75) (xy -0.5 -0.75) (xy 0 -0.75)) (width 0))
+      ))
+    (pad 1 smd custom (at -0.65 0) (size 1 0.5) (layers B.Cu B.Mask)
+      (net 24 "Net-(JP1-Pad1)") (zone_connect 2)
+      (options (clearance outline) (anchor rect))
+      (primitives
+        (gr_circle (center 0 -0.25) (end 0.5 -0.25) (width 0))
+        (gr_circle (center 0 0.25) (end 0.5 0.25) (width 0))
+        (gr_poly (pts
+           (xy 0 0.75) (xy 0.5 0.75) (xy 0.5 -0.75) (xy 0 -0.75)) (width 0))
+      ))
+  )
   (module SirBoardLibrary:SIM28M (layer F.Cu)
     (at 68.2625 41.783 180)
@@
     (tags "Integrated Circuit")
     (attr smd)
-    (fp_text reference SirBoard (at 4.85 5.05 90) (layer F.SilkS)
+    (fp_text reference SIM28M (at 4.85 5.05 90) (layer F.SilkS)
       (effects (font (size 1.27 1.27) (thickness 0.254)))
     )
@@
     (pad 1 thru_hole circle (at 0 0 270) (size 4.5 4.5) (drill 2.7) (layers *.Cu *.Mask))
   )
-  (module MountingHole:MountingHole_2.7mm_M2.5_ISO14580_Pad (layer F.Cu)
-    (at 54.61 44.45 270)
-    (descr "Mounting Hole 2.7mm, M2.5, ISO14580")
-    (tags "mounting hole 2.7mm m2.5 iso14580")
-    (attr virtual)
-    (fp_text reference H1 (at 0 0 90) (layer F.SilkS) hide
-      (effects (font (size 1 1) (thickness 0.15)))
-    )
-    (fp_text value MountingHole (at 0 3.25 90) (layer F.Fab)
-      (effects (font (size 1 1) (thickness 0.15)))
-    )
-    (fp_circle (center 0 0) (end 2.5 0) (layer F.CrtYd) (width 0.05))
-    (fp_circle (center 0 0) (end 2.25 0) (layer Cmts.User) (width 0.15))
-    (fp_text user %R (at 0.3 0 90) (layer F.Fab)
-      (effects (font (size 1 1) (thickness 0.15)))
-    )
-    (pad 1 thru_hole circle (at 0 0 270) (size 4.5 4.5) (drill 2.7) (layers *.Cu *.Mask))
-  )
   (module Capacitor_SMD:C_0805_2012Metric (layer F.Cu)
     (at 71.501 33.2105)
@@
     )
     (pad 1 smd roundrect (at -0.7875 0 90) (size 0.875 0.95) (layers F.Cu F.Paste F.Mask) (roundrect_rratio 0.25)
-      (net 6 "Net-(AE1-Pad1)"))
+      (net 24 "Net-(JP1-Pad1)"))
     (pad 2 smd roundrect (at 0.7875 0 90) (size 0.875 0.95) (layers F.Cu F.Paste F.Mask) (roundrect_rratio 0.25)
       (net 2 "Net-(L1-Pad2)"))
@@
     (tags "Keystone type 3000 coin cell retainer")
     (attr smd)
-    (fp_text reference BT1 (at 0 8) (layer B.SilkS)
+    (fp_text reference CR1220 (at 0 3.937 180 unlocked) (layer B.SilkS)
       (effects (font (size 1 1) (thickness 0.15)) (justify mirror))
     )
@@
     (tags "Hirose U.FL Coaxial")
     (attr smd)
-    (fp_text reference GPS (at 1.016 0 270) (layer F.SilkS) hide
+    (fp_text reference AE1 (at 1.016 0 270) (layer F.SilkS) hide
       (effects (font (size 1 1) (thickness 0.15)))
     )
@@
       (rotate (xyz 0 0 0))
     )
+  )
+  (gr_text "SIM28M\nwww.SirBoard.com" (at 63.5 31.242 180) (layer B.SilkS)
+    (effects (font (size 1 0.9) (thickness 0.15)) (justify mirror))
   )
   (dimension 20.32 (width 0.15) (layer Dwgs.User)
@@
   (segment (start 55.1305 37.046) (end 54.8005 37.046) (width 0.25) (layer F.Cu) (net 6))
   (segment (start 56.4515 35.725) (end 55.1305 37.046) (width 0.25) (layer F.Cu) (net 6))
-  (segment (start 54.14 37.046) (end 54.8005 37.046) (width 0.25) (layer F.Cu) (net 6))
-  (segment (start 53.848 37.338) (end 54.14 37.046) (width 0.25) (layer F.Cu) (net 6))
-  (segment (start 53.1495 37.3) (end 53.1875 37.338) (width 0.25) (layer F.Cu) (net 6))
-  (segment (start 53.1875 37.338) (end 53.848 37.338) (width 0.25) (layer F.Cu) (net 6))
+  (via (at 54.991 39.1795) (size 0.6) (drill 0.3) (layers F.Cu B.Cu) (net 6))
+  (segment (start 55.4505 40.513) (end 55.4505 39.639) (width 0.25) (layer B.Cu) (net 6))
+  (segment (start 55.4505 39.639) (end 54.991 39.1795) (width 0.25) (layer B.Cu) (net 6))
+  (segment (start 54.8005 38.989) (end 54.991 39.1795) (width 0.25) (layer F.Cu) (net 6))
+  (segment (start 54.8005 38.6375) (end 54.8005 38.989) (width 0.25) (layer F.Cu) (net 6))
   (segment (start 56.4515 33.998) (end 56.4515 34.29) (width 0.25) (layer F.Cu) (net 7))
   (segment (start 56.4515 33.998) (end 56.426 33.998) (width 0.25) (layer F.Cu) (net 7))
@@
   (segment (start 58.3565 44.454419) (end 58.3565 45.6565) (width 0.6) (layer B.Cu) (net 23))
   (segment (start 58.3565 41.8365) (end 58.3565 44.454419) (width 0.6) (layer B.Cu) (net 23))
-  (segment (start 55.5365 39.0165) (end 58.3565 41.8365) (width 0.6) (layer B.Cu) (net 23))
-  (segment (start 55.5365 36.7665) (end 55.5365 39.0165) (width 0.6) (layer B.Cu) (net 23))
+  (segment (start 58.3565 37.465) (end 58.3565 41.8365) (width 0.6) (layer B.Cu) (net 23))
+  (segment (start 55.5365 36.7665) (end 57.658 36.7665) (width 0.6) (layer B.Cu) (net 23))
+  (segment (start 57.658 36.7665) (end 58.3565 37.465) (width 0.6) (layer B.Cu) (net 23))
+  (segment (start 68.8975 36.7665) (end 71.3365 36.7665) (width 0.6) (layer B.Cu) (net 23))
+  (segment (start 68.326 37.338) (end 68.8975 36.7665) (width 0.6) (layer B.Cu) (net 23))
+  (segment (start 68.326 40.3225) (end 68.326 37.338) (width 0.6) (layer B.Cu) (net 23))
+  (segment (start 58.3565 41.8365) (end 66.812 41.8365) (width 0.6) (layer B.Cu) (net 23))
+  (segment (start 66.812 41.8365) (end 68.326 40.3225) (width 0.6) (layer B.Cu) (net 23))
   (segment (start 68.272 35.6235) (end 68.2625 35.633) (width 0.25) (layer F.Cu) (net 23))
   (segment (start 69.596 35.6235) (end 68.272 35.6235) (width 0.25) (layer F.Cu) (net 23))
-  (segment (start 71.501 36.0045) (end 69.977 36.0045) (width 0.25) (layer F.Cu) (net 23))
-  (segment (start 69.977 36.0045) (end 69.596 35.6235) (width 0.25) (layer F.Cu) (net 23))
-  (segment (start 71.3365 37.2485) (end 71.3365 36.7665) (width 0.6) (layer B.Cu) (net 23))
-  (segment (start 58.3565 41.8365) (end 66.7485 41.8365) (width 0.6) (layer B.Cu) (net 23))
-  (segment (start 66.7485 41.8365) (end 71.3365 37.2485) (width 0.6) (layer B.Cu) (net 23))
+  (segment (start 70.104 36.1315) (end 69.596 35.6235) (width 0.25) (layer F.Cu) (net 23))
+  (segment (start 71.501 36.0045) (end 71.374 36.1315) (width 0.25) (layer F.Cu) (net 23))
+  (segment (start 71.374 36.1315) (end 70.104 36.1315) (width 0.25) (layer F.Cu) (net 23))
+  (segment (start 53.1495 37.3) (end 53.1875 37.338) (width 0.25) (layer F.Cu) (net 24))
+  (via (at 52.6415 38.2905) (size 0.6) (drill 0.3) (layers F.Cu B.Cu) (net 24))
+  (segment (start 54.1505 40.513) (end 52.6415 39.004) (width 0.25) (layer B.Cu) (net 24))
+  (segment (start 52.6415 39.004) (end 52.6415 38.2905) (width 0.25) (layer B.Cu) (net 24))
+  (segment (start 53.1495 37.7825) (end 52.6415 38.2905) (width 0.25) (layer F.Cu) (net 24))
+  (segment (start 53.1495 37.3) (end 53.1495 37.7825) (width 0.25) (layer F.Cu) (net 24))
   (zone (net 1) (net_name GND) (layer F.Cu) (hatch none 0.508)
     (connect_pads (clearance 0.15))
