File: SIM868/SIM868.sch (KiCad schematic (older format))
At the start: 73 parts, among them CN1 10pF, CN2 10pF, CN3 10pF, CN4 33pF, CN5 33pF, CN6 33pF, J1 104239-1430, J2 AudioJack4, J3 Conn_01x02, J4 USB_B_Micro, J5 Conn_01x11, J6 Conn_01x03, Q1 BC847BDW1, Q2 BC847BDW1, SW1 B3U-1000P, U1 SIM868, U2 MCP73831-2-OT

Commit message: Schematic PDF and 3D Renders added
Parts:
- J1: symbol 104239-1430:104239-1430 -> SIM868-rescue:104239-1430-104239-1430
- U1: symbol SIM868:SIM868 -> SIM868-rescue:SIM868-SIM868
Other:
- moved on the sheet: AE3, BT1, C4, C6, C8, C9, CN1, CN2, CN3, CN4, CN5, CN6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
