File: SIM868/SIM868.kicad_pcb (KiCad board)
At the start: 2 copper layers, 38.1 x 38.1 mm, 73 parts, among them CN1 10pF, CN2 10pF, CN3 10pF, CN4 33pF, CN5 33pF, CN6 33pF, J2 AudioJack4, J4 USB_B_Micro, J5 Conn_01x11, J6 Conn_01x03, Q1 BC847BDW1, Q2 BC847BDW1, U1 SIM868, U2 MCP73831-2-OT

Commit message: Soldermask width adjusted
Other:
- rule solder_mask_min_width: 0.1 -> 0.05
Changed lines of the file:
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@@
   )
   (setup
-    (last_trace_width 0.2)
+    (last_trace_width 0.127)
     (user_trace_width 0.127)
     (user_trace_width 0.15)
@@
     (pad_drill 0)
     (pad_to_mask_clearance 0)
-    (solder_mask_min_width 0.1)
+    (solder_mask_min_width 0.05)
     (aux_axis_origin 0 0)
     (visible_elements 7FFFFFFF)
